File: Hardware/Basic/Top/A10N_TOP.sch (EAGLE design)
At the start: 64 parts, among them SW1 SWITCH.MOM, SW2 SWITCH.MOM, U2 NRF52832_MODULE_MDBT42, U4 PCF8523, U5 FT231XS

Commit message: Connected SD Card, LEDs,
Parts:
- removed C2: 1u, LinnesLab-Passives:CAPACITOR0603
- removed U4: PCF8523, LinnesLab-Clocks:PCF8523
- removed XTAL3: 32.7680kHz, LinnesLab-Clocks:CRYSTALECS-.327-12.5-12-C-TR
Connections:
- removed net BATT: R13.1, R14.2
- removed net CD1: SD2.CARD_DETECT
- removed net CHRG.STAT: CHRG2.STAT, R12.1
- removed net CS.OLED: U3./CS
- removed net DC.OLED: U3.DC/I2C_SA0
- removed net N$19: U4.OSCO, XTAL3.1
- removed net N$20: U4.OSCI, XTAL3.2
- removed net RESET.OLED: U3./RES
- removed net SD.CS: SD2.CS
- removed net VBATT: U4.VBAT
- new net A4/BATT_STATUS: R13.1, R14.2, U2.P0.28/AIN4
- new net A6/TIA: U2.P0.30/AIN6
- new net A7/PPG: U2.P0.31/AIN7
- new net D11/SW2: SW2.1, U2.P0.11
- new net D15/SW1: SW1.1, U2.P0.15
- new net D16/CS_OLED: U2.P0.16, U3./CS
- new net D27/CHRG_STATUS: CHRG2.STAT, R12.1, U2.P0.27
- new net D29/LED_CTRL: U2.P0.29/AIN5
- new net D3/RESET_OLED: U2.P0.03/AIN1, U3./RES
- new net D4/DC_OLED: U2.P0.04/AIN2, U3.DC/I2C_SA0
- new net D5/CRD_DETECT: SD2.CARD_DETECT, U2.P0.05/AIN3
- new net D7/SD_CS: SD2.CS, U2.P0.07
- new net N$27: U2.P0.02/AIN0
- net 3.3V: no longer C2.1, U4.VDD
- net GND: now also SW1.3, SW1.4, SW2.3, SW2.4; no longer C2.2, U4.VSS
- net SCL: no longer U4.SCL
- net SDA: no longer U4.SDA
Other:
- note added: "Digital output"
- note added: "FTDI Serial To USB"
- note removed: "Back-up battery if desired"
- note removed: "I2C Address = 0x68h"
- note removed: "Real Time Clock"
- note removed: "Serial To USB"
- moved on the sheet: C10, C11, C20, C21, C5, C6, C8, C9, CHRG2, D4, D5, J2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

Commit message: Added PPG and Bottom Boards
Parts:
- added C2: 1u, LinnesLab-Passives:CAPACITOR0603
- added U4: PCF8523, LinnesLab-Clocks:PCF8523
- added XTAL3: 32.7680kHz, LinnesLab-Clocks:CRYSTALECS-.327-12.5-12-C-TR
Connections:
- removed net SCL: R2.1, U2.P0.26
- removed net SDA: R1.1, U2.P0.25
- new net D25/SDA: R1.1, U2.P0.25, U4.SDA
- new net D26/SCL: R2.1, U2.P0.26, U4.SCL
- new net N$28: U4.OSCO, XTAL3.1
- new net N$29: U4.OSCI, XTAL3.2
- net 3.3V: now also C2.1, U4.VDD
- net GND: now also C2.2, U4.VSS
Other:
- note added: "I2C Address = 0x68h"
- note added: "Real Time Clock"
- moved on the sheet: R1, R2
Changed lines of the file:
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@@
 <part name="GND1" library="LinnesLab-Symbols" deviceset="GND" device=""/>
 <part name="GND2" library="LinnesLab-Symbols" deviceset="GND" device=""/>
+<part name="GND5" library="LinnesLab-Symbols" deviceset="GND" device=""/>
+<part name="GND6" library="LinnesLab-Symbols" deviceset="GND" device=""/>
+<part name="SUPPLY18" library="LinnesLab-Symbols" deviceset="3.3V" device=""/>
+<part name="C2" library="LinnesLab-Passives" deviceset="CAPACITOR" device="0603" package3d_urn="urn:adsk.eagle:package:15661989/2" value="1u"/>
+<part name="SUPPLY19" library="LinnesLab-Symbols" deviceset="3.3V" device=""/>
+<part name="XTAL3" library="LinnesLab-Clocks" deviceset="CRYSTAL" device="ECS-.327-12.5-12-C-TR" package3d_urn="urn:adsk.eagle:package:18579459/2" value="32.7680kHz">
+<attribute name="FREQ" value="32.7680KHZ"/>
+</part>
+<part name="U4" library="LinnesLab-Clocks" deviceset="PCF8523" device="" package3d_urn="urn:adsk.eagle:package:18599600/2">
+<attribute name="DIGIKEY" value="568-5306-1-ND"/>
+<attribute name="I2C_ADDRESS" value="0x68h"/>
+<attribute name="MFN" value="PCF8523T/1,118"/>
+<attribute name="MFN_MANUFACTURER" value="NXP USA Inc."/>
+</part>
 </parts>
 <sheets>
@@
 <text x="363.22" y="-12.7" size="5.08" layer="97">FTDI Serial To USB</text>
 <text x="66.04" y="-78.74" size="1.778" layer="91">Digital output</text>
+<text x="327.66" y="12.7" size="1.27" layer="97">I2C Address = 0x68h</text>
+<text x="297.18" y="40.64" size="5.08" layer="97">Real Time Clock</text>
 </plain>
 <instances>
@@
 <attribute name="VALUE" x="435.61" y="-43.942" size="1.778" layer="96"/>
 </instance>
-<instance part="R1" gate="G$1" x="15.24" y="177.8" smashed="yes" rot="R90">
-<attribute name="NAME" x="13.7414" y="173.99" size="1.778" layer="95" rot="R90"/>
-<attribute name="VALUE" x="18.542" y="173.99" size="1.778" layer="96" rot="R90"/>
-</instance>
-<instance part="R2" gate="G$1" x="25.4" y="177.8" smashed="yes" rot="R90">
-<attribute name="NAME" x="23.9014" y="173.99" size="1.778" layer="95" rot="R90"/>
-<attribute name="VALUE" x="28.702" y="173.99" size="1.778" layer="96" rot="R90"/>
-</instance>
-<instance part="SUPPLY1" gate="G$1" x="15.24" y="185.42" smashed="yes">
-<attribute name="VALUE" x="15.24" y="188.214" size="1.778" layer="96" align="bottom-center"/>
-</instance>
-<instance part="SUPPLY6" gate="G$1" x="25.4" y="185.42" smashed="yes">
-<attribute name="VALUE" x="25.4" y="188.214" size="1.778" layer="96" align="bottom-center"/>
+<instance part="R1" gate="G$1" x="20.32" y="162.56" smashed="yes" rot="R90">
+<attribute name="NAME" x="18.8214" y="158.75" size="1.778" layer="95" rot="R90"/>
+<attribute name="VALUE" x="23.622" y="158.75" size="1.778" layer="96" rot="R90"/>
+</instance>
+<instance part="R2" gate="G$1" x="30.48" y="162.56" smashed="yes" rot="R90">
+<attribute name="NAME" x="28.9814" y="158.75" size="1.778" layer="95" rot="R90"/>
+<attribute name="VALUE" x="33.782" y="158.75" size="1.778" layer="96" rot="R90"/>
+</instance>
+<instance part="SUPPLY1" gate="G$1" x="20.32" y="170.18" smashed="yes">
+<attribute name="VALUE" x="20.32" y="172.974" size="1.778" layer="96" align="bottom-center"/>
+</instance>
+<instance part="SUPPLY6" gate="G$1" x="30.48" y="170.18" smashed="yes">
+<attribute name="VALUE" x="30.48" y="172.974" size="1.778" layer="96" align="bottom-center"/>
 </instance>
 <instance part="GND1" gate="G$1" x="439.42" y="10.16" smashed="yes">
@@
 <instance part="GND2" gate="G$1" x="487.68" y="10.16" smashed="yes">
 <attribute name="VALUE" x="487.68" y="9.906" size="1.778" layer="96" align="top-center"/>
+</instance>
+<instance part="GND5" gate="G$1" x="294.64" y="12.7" smashed="yes">
+<attribute name="VALUE" x="294.64" y="12.446" size="1.778" layer="96" align="top-center"/>
+</instance>
+<instance part="GND6" gate="G$1" x="360.68" y="17.78" smashed="yes">
+<attribute name="VALUE" x="360.68" y="17.526" size="1.778" layer="96" align="top-center"/>
+</instance>
+<instance part="SUPPLY18" gate="G$1" x="330.2" y="27.94" smashed="yes">
+<attribute name="VALUE" x="330.2" y="30.734" size="1.778" layer="96" align="bottom-center"/>
+</instance>
+<instance part="C2" gate="G$1" x="360.68" y="25.4" smashed="yes">
+<attribute name="NAME" x="362.204" y="28.321" size="1.778" layer="95"/>
+<attribute name="VALUE" x="362.204" y="23.241" size="1.778" layer="96"/>
+</instance>
+<instance part="SUPPLY19" gate="G$1" x="360.68" y="33.02" smashed="yes">
+<attribute name="VALUE" x="360.68" y="35.814" size="1.778" layer="96" align="bottom-center"/>
+</instance>
+<instance part="XTAL3" gate="G$1" x="292.1" y="25.4" smashed="yes">
+<attribute name="NAME" x="292.1" y="27.432" size="1.778" layer="95" font="vector" align="bottom-center"/>
+<attribute name="FREQ" x="292.1" y="25.4" size="1.27" layer="96" display="off"/>
+</instance>
+<instance part="U4" gate="G$1" x="312.42" y="22.86" smashed="yes">
+<attribute name="NAME" x="299.72" y="29.21" size="1.778" layer="95"/>
+<attribute name="VALUE" x="299.72" y="12.7" size="1.778" layer="96"/>
+<attribute name="DIGIKEY" x="312.42" y="22.86" size="1.27" layer="96" display="off"/>
+<attribute name="I2C_ADDRESS" x="312.42" y="22.86" size="1.27" layer="96" display="off"/>
+<attribute name="MFN" x="312.42" y="22.86" size="1.27" layer="96" display="off"/>
+<attribute name="MFN_MANUFACTURER" x="312.42" y="22.86" size="1.27" layer="96" display="off"/>
 </instance>
 </instances>
@@
 <pinref part="GND2" gate="G$1" pin="GND"/>
 </segment>
+<segment>
+<wire x1="297.18" y1="17.78" x2="294.64" y2="17.78" width="0.1524" layer="91"/>
+<wire x1="294.64" y1="15.24" x2="294.64" y2="17.78" width="0.1524" layer="91"/>
+<pinref part="GND5" gate="G$1" pin="GND"/>
+<pinref part="U4" gate="G$1" pin="VSS"/>
+</segment>
+<segment>
+<wire x1="360.68" y1="20.32" x2="360.68" y2="22.86" width="0.1524" layer="91"/>
+<pinref part="GND6" gate="G$1" pin="GND"/>
+<pinref part="C2" gate="G$1" pin="2"/>
+</segment>
 </net>
 <net name="SWDIO" class="0">
@@
 <pinref part="R1" gate="G$1" pin="2"/>
 <pinref part="SUPPLY1" gate="G$1" pin="3.3V"/>
-<wire x1="15.24" y1="185.42" x2="15.24" y2="182.88" width="0.1524" layer="91"/>
+<wire x1="20.32" y1="170.18" x2="20.32" y2="167.64" width="0.1524" layer="91"/>
 </segment>
 <segment>
 <pinref part="R2" gate="G$1" pin="2"/>
 <pinref part="SUPPLY6" gate="G$1" pin="3.3V"/>
-<wire x1="25.4" y1="185.42" x2="25.4" y2="182.88" width="0.1524" layer="91"/>
-</segment>
-</net>
-<net name="SDA" class="0">
+<wire x1="30.48" y1="170.18" x2="30.48" y2="167.64" width="0.1524" layer="91"/>
+</segment>
+<segment>
+<wire x1="327.66" y1="25.4" x2="330.2" y2="25.4" width="0.1524" layer="91"/>
+<wire x1="330.2" y1="27.94" x2="330.2" y2="25.4" width="0.1524" layer="91"/>
+<pinref part="SUPPLY18" gate="G$1" pin="3.3V"/>
+<pinref part="U4" gate="G$1" pin="VDD"/>
+</segment>
+<segment>
+<pinref part="C2" gate="G$1" pin="1"/>
+<pinref part="SUPPLY19" gate="G$1" pin="3.3V"/>
+<wire x1="360.68" y1="33.02" x2="360.68" y2="30.48" width="0.1524" layer="91"/>
+</segment>
+</net>
+<net name="D25/SDA" class="0">
 <segment>
 <wire x1="76.2" y1="152.4" x2="73.66" y2="152.4" width="0.1524" layer="91"/>
@@
 <segment>
 <pinref part="R1" gate="G$1" pin="1"/>
-<wire x1="15.24" y1="172.72" x2="15.24" y2="170.18" width="0.1524" layer="91"/>
-<label x="15.24" y="170.18" size="1.778" layer="95" rot="R180" xref="yes"/>
-</segment>
-</net>
-<net name="SCL" class="0">
+<wire x1="20.32" y1="157.48" x2="20.32" y2="154.94" width="0.1524" layer="91"/>
+<label x="20.32" y="154.94" size="1.778" layer="95" rot="R180" xref="yes"/>
+</segment>
+<segment>
+<wire x1="327.66" y1="17.78" x2="332.74" y2="17.78" width="0.1524" layer="91"/>
+<label x="332.74" y="17.78" size="1.27" layer="95" xref="yes"/>
+<pinref part="U4" gate="G$1" pin="SDA"/>
+</segment>
+</net>
+<net name="D26/SCL" class="0">
 <segment>
 <wire x1="76.2" y1="149.86" x2="73.66" y2="149.86" width="0.1524" layer="91"/>
@@
 <segment>
 <pinref part="R2" gate="G$1" pin="1"/>
-<wire x1="25.4" y1="172.72" x2="25.4" y2="170.18" width="0.1524" layer="91"/>
-<label x="25.4" y="170.18" size="1.778" layer="95" xref="yes"/>
+<wire x1="30.48" y1="157.48" x2="30.48" y2="154.94" width="0.1524" layer="91"/>
+<label x="30.48" y="154.94" size="1.778" layer="95" xref="yes"/>
+</segment>
+<segment>
+<label x="332.74" y="20.32" size="1.27" layer="95" xref="yes"/>
+<wire x1="327.66" y1="20.32" x2="332.74" y2="20.32" width="0.1524" layer="91"/>
+<pinref part="U4" gate="G$1" pin="SCL"/>
 </segment>
 </net>
@@
 </segment>
 </net>
+<net name="N$28" class="0">
+<segment>
+<wire x1="297.18" y1="22.86" x2="287.02" y2="22.86" width="0.1524" layer="91"/>
+<wire x1="287.02" y1="22.86" x2="287.02" y2="25.4" width="0.1524" layer="91"/>
+<wire x1="287.02" y1="25.4" x2="289.56" y2="25.4" width="0.1524" layer="91"/>
+<pinref part="XTAL3" gate="G$1" pin="1"/>
+<pinref part="U4" gate="G$1" pin="OSCO"/>
+</segment>
+</net>
+<net name="N$29" class="0">
+<segment>
+<wire x1="294.64" y1="25.4" x2="297.18" y2="25.4" width="0.1524" layer="91"/>
+<pinref part="XTAL3" gate="G$1" pin="2"/>
+<pinref part="U4" gate="G$1" pin="OSCI"/>
+</segment>
+</net>
